Commit message: added roughybot_description package. changed robot_core.urdf.xacro: made adding camera and lidar conditional. added view_roughybot.launch.py

File: src/roughybot_description/urdf/robot_core.urdf.xacro (robot description, xacro)
@@ -1,4 +1,4 @@
 <?xml version="1.0" ?>
-<robot name="roughybot_sim" xmlns:xacro="http://www.ros.org/wiki/xacro">
+<robot name="roughybot" xmlns:xacro="http://www.ros.org/wiki/xacro">
     <xacro:property name="base_mass" value="1.5"/>
     <xacro:property name="base_length" value="0.508"/>
@@ -12,6 +12,8 @@
     <xacro:include filename="inertial_macros.urdf.xacro"/>
     <xacro:include filename="material.urdf.xacro"/>
+    <xacro:include filename="gazebo_params.gazebo"/>
     <xacro:include filename="ros2_control.urdf.xacro"/>
-    <xacro:include filename="gazebo_params.gazebo"/>
+    <xacro:arg name="add_camera" default="true"/>
+    <xacro:arg name="add_lidar" default="true"/>
     <link name="base_footprint">
     </link>
@@ -28,5 +30,5 @@
             <origin xyz="0 0 0" rpy="0 0 0"/>
             <geometry>
-                <mesh filename="package://roughybot_sim/robot_description/meshes/base_link.stl" scale="0.001 0.001 0.001"/>
+                <mesh filename="package://roughybot_description/meshes/base_link.stl" scale="0.001 0.001 0.001"/>
                 <!-- <box size="${base_length} ${base_width} ${base_height}"/> -->
             </geometry>
@@ -36,5 +38,5 @@
             <origin xyz="0 0 0" rpy="0 0 0"/>
             <geometry>
-                <mesh filename="package://roughybot_sim/robot_description/meshes/base_link.stl" scale="0.001 0.001 0.001"/>
+                <mesh filename="package://roughybot_description/meshes/base_link.stl" scale="0.001 0.001 0.001"/>
             </geometry>
         </collision>
@@ -54,5 +56,5 @@
             <origin xyz="0.214 0.1651 -0.040" rpy="0 0 0"/>
             <geometry>
-                <mesh filename="package://roughybot_sim/robot_description/meshes/right_wheel_link.stl" scale="0.001 0.001 0.001"/>
+                <mesh filename="package://roughybot_description/meshes/right_wheel_link.stl" scale="0.001 0.001 0.001"/>
                 <!-- <cylinder radius="${wheel_radius}" length="${wheel_length}"/> -->
             </geometry>
@@ -62,5 +64,5 @@
             <origin xyz="0.214 0.1651 -0.040" rpy="0 0 0"/>
             <geometry>
-                <mesh filename="package://roughybot_sim/robot_description/meshes/right_wheel_link.stl" scale="0.001 0.001 0.001"/>
+                <mesh filename="package://roughybot_description/meshes/right_wheel_link.stl" scale="0.001 0.001 0.001"/>
             </geometry>
         </collision>
@@ -80,5 +82,5 @@
             <origin xyz="0.214 -0.1651 -0.040" rpy="0 0 0"/>
             <geometry>
-                <mesh filename="package://roughybot_sim/robot_description/meshes/left_wheel_link.stl" scale="0.001 0.001 0.001"/>
+                <mesh filename="package://roughybot_description/meshes/left_wheel_link.stl" scale="0.001 0.001 0.001"/>
                 <!-- <cylinder radius="${wheel_radius}" length="${wheel_length}"/> -->
             </geometry>
@@ -88,5 +90,5 @@
             <origin xyz="0.214 -0.1651 -0.040" rpy="0 0 0"/>
             <geometry>
-                <mesh filename="package://roughybot_sim/robot_description/meshes/left_wheel_link.stl" scale="0.001 0.001 0.001"/>
+                <mesh filename="package://roughybot_description/meshes/left_wheel_link.stl" scale="0.001 0.001 0.001"/>
             </geometry>
         </collision>
@@ -117,50 +119,61 @@
     </link>
     <!-- CAMERA LINK -->
-    <joint name="camera_joint" type="fixed">
-        <origin xyz="0.264 0 0.080" rpy="0 0 0"/>
-        <parent link="base_link"/>
-        <child link="camera_link"/>
-    </joint>
-    <link name="camera_link">
-        <xacro:inertial_box mass="${camera_mass}" x="0.025" y="0.088" z="0.021">
-            <origin xyz="0 0 0" rpy="0 0 1.57"/>
-        </xacro:inertial_box>
-        <visual>
-            <origin xyz="0 0 0" rpy="0 0 1.57"/>
-            <geometry>
-                <mesh filename="package://roughybot_sim/robot_description/meshes/camera_link.stl" scale="0.001 0.001 0.001"/>
-            </geometry>
-            <material name="lidar_color"/>
-        </visual>
-        <collision>
-            <origin xyz="0 0 0" rpy="0 0 1.57"/>
-            <geometry>
-                <mesh filename="package://roughybot_sim/robot_description/meshes/camera_link.stl" scale="0.001 0.001 0.001"/>
-            </geometry>
-        </collision>
-    </link>
+    <xacro:if value="$(arg add_camera)">
+        <joint name="camera_joint" type="fixed">
+            <origin xyz="0.264 0 0.080" rpy="0 0 0"/>
+            <parent link="base_link"/>
+            <child link="camera_link"/>
+        </joint>
+        <link name="camera_link">
+            <xacro:inertial_box mass="${camera_mass}" x="0.025" y="0.088" z="0.021">
+                <origin xyz="0 0 0" rpy="0 0 1.57"/>
+            </xacro:inertial_box>
+            <visual>
+                <origin xyz="0 0 0" rpy="0 0 1.57"/>
+                <geometry>
+                    <mesh filename="package://roughybot_description/meshes/camera_link.stl" scale="0.001 0.001 0.001"/>
+                </geometry>
+                <material name="lidar_color"/>
+            </visual>
+            <collision>
+                <origin xyz="0 0 0" rpy="0 0 1.57"/>
+                <geometry>
+                    <mesh filename="package://roughybot_description/meshes/camera_link.stl" scale="0.001 0.001 0.001"/>
+                </geometry>
+            </collision>
+        </link>
+        <joint name="optical_joint" type="fixed">
+            <parent link="camera_link"/>
+            <child link="optical_link"/>
+            <origin xyz="0 0 0" rpy="-1.57 0 -1.57"/>
+        </joint>
+        <link name="optical_link">
+        </link>
+    </xacro:if>
     <!-- LIDAR LINK -->
-    <joint name="lidar_joint" type="fixed">
-        <origin xyz="0.210 0 0.1016" rpy="0 0 0"/>
-        <parent link="base_link"/>
-        <child link="lidar_link"/>
-    </joint>
-    <link name="lidar_link">
-        <xacro:inertial_cylinder mass="${lidar_mass}" length="0.08" radius="0.052">
-            <origin xyz="0 0 0" rpy="0 0 0"/>
-        </xacro:inertial_cylinder>
-        <visual>
-            <origin xyz="0 0 0" rpy="0 0 0"/>
-            <geometry>
-                <mesh filename="package://roughybot_sim/robot_description/meshes/lidar_link.stl" scale="0.001 0.001 0.001"/>
-            </geometry>
-            <material name="lidar_color"/>
-        </visual>
-        <collision>
-            <origin xyz="0 0 0" rpy="0 0 0"/>
-            <geometry>
-                <mesh filename="package://roughybot_sim/robot_description/meshes/lidar_link.stl" scale="0.001 0.001 0.001"/>
-            </geometry>
-        </collision>
-    </link>
+    <xacro:if value="$(arg add_lidar)">
+        <joint name="lidar_joint" type="fixed">
+            <origin xyz="0.20 0 0.1016" rpy="0 0 0"/>
+            <parent link="base_link"/>
+            <child link="lidar_link"/>
+        </joint>
+        <link name="lidar_link">
+            <xacro:inertial_cylinder mass="${lidar_mass}" length="0.08" radius="0.052">
+                <origin xyz="0 0 0" rpy="0 0 0"/>
+            </xacro:inertial_cylinder>
+            <visual>
+                <origin xyz="0 0 0" rpy="0 0 0"/>
+                <geometry>
+                    <mesh filename="package://roughybot_description/meshes/lidar_link.stl" scale="0.001 0.001 0.001"/>
+                </geometry>
+                <material name="lidar_color"/>
+            </visual>
+            <collision>
+                <origin xyz="0 0 0" rpy="0 0 0"/>
+                <geometry>
+                    <mesh filename="package://roughybot_description/meshes/lidar_link.stl" scale="0.001 0.001 0.001"/>
+                </geometry>
+            </collision>
+        </link>
+    </xacro:if>
 </robot>

File: src/roughybot_description/urdf/ros2_control.urdf.xacro (robot description, xacro)
@@ -24,5 +24,5 @@
     <gazebo>
         <plugin filename="gz_ros2_control-system" name="gz_ros2_control::GazeboSimROS2ControlPlugin">
-            <parameters>$(find roughybot_sim)/config/controller_config.yaml</parameters>
+            <parameters>package://roughybot_description/config/controller_config.yaml</parameters>
         </plugin>
     </gazebo>

Commit message: fixed launch files

File: src/roughybot_description/urdf/robot_core.urdf.xacro (robot description, xacro)
@@ -154,5 +154,5 @@
     <xacro:if value="$(arg add_lidar)">
         <joint name="lidar_joint" type="fixed">
-            <origin xyz="0.20 0 0.1016" rpy="0 0 0"/>
+            <origin xyz="0.210 0 0.1016" rpy="0 0 0"/>
             <parent link="base_link"/>
             <child link="lidar_link"/>

File: src/roughybot_description/urdf/ros2_control.urdf.xacro (robot description, xacro)
@@ -24,5 +24,5 @@
     <gazebo>
         <plugin filename="gz_ros2_control-system" name="gz_ros2_control::GazeboSimROS2ControlPlugin">
-            <parameters>package://roughybot_description/config/controller_config.yaml</parameters>
+            <parameters>$(find roughybot_description)/config/controller_config.yaml</parameters>
         </plugin>
     </gazebo>
